File: PCB/Flightime.kicad_pcb (KiCad board)
At the start: 2 copper layers, 61.8 x 36.8 mm, 30 parts, among them J1 JST_02, J2 JST_02, J3 JST_02, J4 JST_02, J5 Conn_01x02_Pin, J6 Conn_01x02_Pin, Q1 AO3400A, Q2 AO3400A, Q3 AO3400A, Q4 AO3400A, SW1 SW_Nidec_CAS-120A1, U1 XIAO-ESP32-S3-SMD, U2 GY-521

Commit message: reorientazted s3
Parts:
- moved U1 28.0 mm to (141.1, 82.9), turned to -90 degrees
Routing:
- net Net-(U1-D4): track 78.2 -> 114.8 mm, vias 0 -> 2
- net Net-(U1-D5): track 74.1 -> 110.0 mm
- net 3.3V: track 68.6 -> 104.2 mm
- net Net-(U1-D3): track 6.99 -> 36.8 mm, vias 0 -> 2
- net Net-(U1-D10): track 50.8 -> 79.1 mm, vias 3 -> 5
- net Net-(U1-D0): track 3.98 -> 29.2 mm, vias 0 -> 2
- net Net-(U1-D1): track 4.95 -> 25.8 mm, vias 0 -> 2
- net Net-(U1-D2): track 6.19 -> 26.5 mm, vias 0 -> 4
- net GND: track 115.6 -> 120.1 mm
- net -BATT: track 55.7 -> 53.4 mm, vias 1 -> 3
- net +BATT: track 85.1 -> 87.4 mm
Other:
- board size 61.8 x 36.8 mm -> 61.8 x 38.8 mm
